Commit message: use relative paths

File: urdf/stationary_ai.urdf (robot description, URDF)
Before this commit: robot stationary_ai, 70 links, 69 joints
Links:
- link cam_high_link: geometry collision box size=0.023 0.042 0.042; visual mesh filename=../meshes/peripherals/d405.stl scale=0.001 0.001 0.001
- link cam_high_mount_link: geometry collision mesh filename=../meshes/stationary_ai/cam_high_mount_link.stl; visual mesh filename=../meshes/stationary_ai/cam_high_mount_link.stl
- link cam_low_link: geometry collision box size=0.023 0.042 0.042; visual mesh filename=../meshes/peripherals/d405.stl scale=0.001 0.001 0.001
- link cam_low_mount_link: geometry collision mesh filename=../meshes/stationary_ai/cam_low_mount_link.stl; visual mesh filename=../meshes/stationary_ai/cam_low_mount_link.stl
- link follower_left_base_link: geometry collision mesh filename=../meshes/wxai/base_link.stl; visual mesh filename=../meshes/wxai/base_link.stl
- link follower_left_camera_link: geometry collision box size=0.023 0.042 0.042; visual mesh filename=../meshes/peripherals/d405.stl scale=0.001 0.001 0.001
- link follower_left_camera_mount_d405: geometry collision mesh filename=../meshes/wxai/camera_mount_d405.stl; visual mesh filename=../meshes/wxai/camera_mount_d405.stl
- link follower_left_carriage_left: geometry collision mesh filename=../meshes/wxai/carriage_left.stl; visual mesh filename=../meshes/wxai/carriage_left.stl
- link follower_left_carriage_right: geometry collision mesh filename=../meshes/wxai/carriage_right.stl; visual mesh filename=../meshes/wxai/carriage_right.stl
- link follower_left_gripper_left: geometry collision mesh filename=../meshes/wxai/gripper_left.stl; visual mesh filename=../meshes/wxai/gripper_left.stl
- link follower_left_gripper_right: geometry collision mesh filename=../meshes/wxai/gripper_right.stl; visual mesh filename=../meshes/wxai/gripper_right.stl
- link follower_left_link_1: geometry collision mesh filename=../meshes/wxai/link_1.stl; visual mesh filename=../meshes/wxai/link_1.stl
- link follower_left_link_2: geometry collision mesh filename=../meshes/wxai/link_2.stl; visual mesh filename=../meshes/wxai/link_2.stl
- link follower_left_link_3: geometry collision mesh filename=../meshes/wxai/link_3.stl; visual mesh filename=../meshes/wxai/link_3.stl
- link follower_left_link_4: geometry collision mesh filename=../meshes/wxai/link_4.stl; visual mesh filename=../meshes/wxai/link_4.stl
- link follower_left_link_5: geometry collision mesh filename=../meshes/wxai/link_5.stl; visual mesh filename=../meshes/wxai/link_5.stl
- link follower_left_link_6: geometry collision mesh filename=../meshes/wxai/link_6.stl; visual mesh filename=../meshes/wxai/link_6.stl
- link follower_right_base_link: geometry collision mesh filename=../meshes/wxai/base_link.stl; visual mesh filename=../meshes/wxai/base_link.stl
- link follower_right_camera_link: geometry collision box size=0.023 0.042 0.042; visual mesh filename=../meshes/peripherals/d405.stl scale=0.001 0.001 0.001
- link follower_right_camera_mount_d405: geometry collision mesh filename=../meshes/wxai/camera_mount_d405.stl; visual mesh filename=../meshes/wxai/camera_mount_d405.stl
- link follower_right_carriage_left: geometry collision mesh filename=../meshes/wxai/carriage_left.stl; visual mesh filename=../meshes/wxai/carriage_left.stl
- link follower_right_carriage_right: geometry collision mesh filename=../meshes/wxai/carriage_right.stl; visual mesh filename=../meshes/wxai/carriage_right.stl
- link follower_right_gripper_left: geometry collision mesh filename=../meshes/wxai/gripper_left.stl; visual mesh filename=../meshes/wxai/gripper_left.stl
- link follower_right_gripper_right: geometry collision mesh filename=../meshes/wxai/gripper_right.stl; visual mesh filename=../meshes/wxai/gripper_right.stl
- link follower_right_link_1: geometry collision mesh filename=../meshes/wxai/link_1.stl; visual mesh filename=../meshes/wxai/link_1.stl
- link follower_right_link_2: geometry collision mesh filename=../meshes/wxai/link_2.stl; visual mesh filename=../meshes/wxai/link_2.stl
- link follower_right_link_3: geometry collision mesh filename=../meshes/wxai/link_3.stl; visual mesh filename=../meshes/wxai/link_3.stl
- link follower_right_link_4: geometry collision mesh filename=../meshes/wxai/link_4.stl; visual mesh filename=../meshes/wxai/link_4.stl
- link follower_right_link_5: geometry collision mesh filename=../meshes/wxai/link_5.stl; visual mesh filename=../meshes/wxai/link_5.stl
- link follower_right_link_6: geometry collision mesh filename=../meshes/wxai/link_6.stl; visual mesh filename=../meshes/wxai/link_6.stl
- link frame_link: geometry collision mesh filename=../meshes/stationary_ai/frame_link.stl; visual mesh filename=../meshes/stationary_ai/frame_link.stl
- link tabletop_link: geometry collision mesh filename=../meshes/stationary_ai/tabletop_link.stl; visual mesh filename=../meshes/stationary_ai/tabletop_link.stl

Commit message: convert stl to obj with meshlab

File: urdf/stationary_ai.urdf (robot description, URDF)
Before this commit: robot stationary_ai, 70 links, 69 joints
Links:
- link cam_high_link: geometry collision box size=0.023 0.042 0.042; visual mesh filename=../meshes/peripherals/d405.obj scale=0.001 0.001 0.001
- link cam_high_mount_link: geometry collision mesh filename=../meshes/stationary_ai/cam_high_mount_link.obj; visual mesh filename=../meshes/stationary_ai/cam_high_mount_link.obj
- link cam_low_link: geometry collision box size=0.023 0.042 0.042; visual mesh filename=../meshes/peripherals/d405.obj scale=0.001 0.001 0.001
- link cam_low_mount_link: geometry collision mesh filename=../meshes/stationary_ai/cam_low_mount_link.obj; visual mesh filename=../meshes/stationary_ai/cam_low_mount_link.obj
- link follower_left_base_link: geometry collision mesh filename=../meshes/wxai/base_link.obj; visual mesh filename=../meshes/wxai/base_link.obj
- link follower_left_camera_link: geometry collision box size=0.023 0.042 0.042; visual mesh filename=../meshes/peripherals/d405.obj scale=0.001 0.001 0.001
- link follower_left_camera_mount_d405: geometry collision mesh filename=../meshes/wxai/camera_mount_d405.obj; visual mesh filename=../meshes/wxai/camera_mount_d405.obj
- link follower_left_carriage_left: geometry collision mesh filename=../meshes/wxai/carriage_left.obj; visual mesh filename=../meshes/wxai/carriage_left.obj
- link follower_left_carriage_right: geometry collision mesh filename=../meshes/wxai/carriage_right.obj; visual mesh filename=../meshes/wxai/carriage_right.obj
- link follower_left_gripper_left: geometry collision mesh filename=../meshes/wxai/gripper_left.obj; visual mesh filename=../meshes/wxai/gripper_left.obj
- link follower_left_gripper_right: geometry collision mesh filename=../meshes/wxai/gripper_right.obj; visual mesh filename=../meshes/wxai/gripper_right.obj
- link follower_left_link_1: geometry collision mesh filename=../meshes/wxai/link_1.obj; visual mesh filename=../meshes/wxai/link_1.obj
- link follower_left_link_2: geometry collision mesh filename=../meshes/wxai/link_2.obj; visual mesh filename=../meshes/wxai/link_2.obj
- link follower_left_link_3: geometry collision mesh filename=../meshes/wxai/link_3.obj; visual mesh filename=../meshes/wxai/link_3.obj
- link follower_left_link_4: geometry collision mesh filename=../meshes/wxai/link_4.obj; visual mesh filename=../meshes/wxai/link_4.obj
- link follower_left_link_5: geometry collision mesh filename=../meshes/wxai/link_5.obj; visual mesh filename=../meshes/wxai/link_5.obj
- link follower_left_link_6: geometry collision mesh filename=../meshes/wxai/link_6.obj; visual mesh filename=../meshes/wxai/link_6.obj
- link follower_right_base_link: geometry collision mesh filename=../meshes/wxai/base_link.obj; visual mesh filename=../meshes/wxai/base_link.obj
- link follower_right_camera_link: geometry collision box size=0.023 0.042 0.042; visual mesh filename=../meshes/peripherals/d405.obj scale=0.001 0.001 0.001
- link follower_right_camera_mount_d405: geometry collision mesh filename=../meshes/wxai/camera_mount_d405.obj; visual mesh filename=../meshes/wxai/camera_mount_d405.obj
- link follower_right_carriage_left: geometry collision mesh filename=../meshes/wxai/carriage_left.obj; visual mesh filename=../meshes/wxai/carriage_left.obj
- link follower_right_carriage_right: geometry collision mesh filename=../meshes/wxai/carriage_right.obj; visual mesh filename=../meshes/wxai/carriage_right.obj
- link follower_right_gripper_left: geometry collision mesh filename=../meshes/wxai/gripper_left.obj; visual mesh filename=../meshes/wxai/gripper_left.obj
- link follower_right_gripper_right: geometry collision mesh filename=../meshes/wxai/gripper_right.obj; visual mesh filename=../meshes/wxai/gripper_right.obj
- link follower_right_link_1: geometry collision mesh filename=../meshes/wxai/link_1.obj; visual mesh filename=../meshes/wxai/link_1.obj
- link follower_right_link_2: geometry collision mesh filename=../meshes/wxai/link_2.obj; visual mesh filename=../meshes/wxai/link_2.obj
- link follower_right_link_3: geometry collision mesh filename=../meshes/wxai/link_3.obj; visual mesh filename=../meshes/wxai/link_3.obj
- link follower_right_link_4: geometry collision mesh filename=../meshes/wxai/link_4.obj; visual mesh filename=../meshes/wxai/link_4.obj
- link follower_right_link_5: geometry collision mesh filename=../meshes/wxai/link_5.obj; visual mesh filename=../meshes/wxai/link_5.obj
- link follower_right_link_6: geometry collision mesh filename=../meshes/wxai/link_6.obj; visual mesh filename=../meshes/wxai/link_6.obj
- link frame_link: geometry collision mesh filename=../meshes/stationary_ai/frame_link.obj; visual mesh filename=../meshes/stationary_ai/frame_link.obj
- link tabletop_link: geometry collision mesh filename=../meshes/stationary_ai/tabletop_link.obj; visual mesh filename=../meshes/stationary_ai/tabletop_link.obj

Commit message: simplify tabletop collision geom

File: urdf/stationary_ai.urdf (robot description, URDF)
Before this commit: robot stationary_ai, 70 links, 69 joints
Links:
- link tabletop_link: geometry collision box size=0.749 1.2192 0.02; visual mesh filename=../meshes/stationary_ai/tabletop_link.obj

Commit message: replace frame with primitive geometries

File: urdf/stationary_ai.urdf (robot description, URDF)
Before this commit: robot stationary_ai, 70 links, 69 joints
Links:
- link frame_link: geometry collision box size=0.02 0.02 0.35; collision box size=0.02 0.02 0.35

Commit message: exclude camera mounts from collision geometry

File: urdf/stationary_ai.urdf (robot description, URDF)
Before this commit: robot stationary_ai, 70 links, 69 joints
Links:
- link cam_high_mount_link: geometry visual mesh filename=../meshes/stationary_ai/cam_high_mount_link.obj
- link cam_low_mount_link: geometry visual mesh filename=../meshes/stationary_ai/cam_low_mount_link.obj

Commit message: simplify left arm collision geometries

File: urdf/stationary_ai.urdf (robot description, URDF)
Before this commit: robot stationary_ai, 70 links, 69 joints
Links:
- link follower_left_base_link: geometry collision cylinder length=0.055 radius=0.034; visual mesh filename=../meshes/wxai/base_link.obj
- link follower_left_camera_link: geometry collision box size=0.027 0.045 0.045; visual mesh filename=../meshes/peripherals/d405.obj scale=0.001 0.001 0.001
- link follower_left_camera_mount_d405: geometry visual mesh filename=../meshes/wxai/camera_mount_d405.obj
- link follower_left_carriage_left: geometry visual mesh filename=../meshes/wxai/carriage_left.obj
- link follower_left_carriage_right: geometry visual mesh filename=../meshes/wxai/carriage_right.obj
- link follower_left_link_1: geometry visual mesh filename=../meshes/wxai/link_1.obj
- link follower_left_link_2: geometry collision box size=0.3 0.05 0.05; visual mesh filename=../meshes/wxai/link_2.obj
- link follower_left_link_3: geometry collision box size=0.22 0.05 0.04; visual mesh filename=../meshes/wxai/link_3.obj
- link follower_left_link_4: geometry collision cylinder length=0.06 radius=0.029; visual mesh filename=../meshes/wxai/link_4.obj
- link follower_left_link_5: geometry collision cylinder length=0.05 radius=0.029; visual mesh filename=../meshes/wxai/link_5.obj
- link follower_left_link_6: geometry collision box size=0.025 0.187 0.0618; collision cylinder length=0.05 radius=0.029

Commit message: propagate simplifications to the right arm

File: urdf/stationary_ai.urdf (robot description, URDF)
Before this commit: robot stationary_ai, 70 links, 69 joints
Links:
- link follower_right_base_link: geometry collision cylinder length=0.055 radius=0.034; visual mesh filename=../meshes/wxai/base_link.obj
- link follower_right_camera_link: geometry collision box size=0.027 0.045 0.045; visual mesh filename=../meshes/peripherals/d405.obj scale=0.001 0.001 0.001
- link follower_right_camera_mount_d405: geometry visual mesh filename=../meshes/wxai/camera_mount_d405.obj
- link follower_right_carriage_left: geometry visual mesh filename=../meshes/wxai/carriage_left.obj
- link follower_right_carriage_right: geometry visual mesh filename=../meshes/wxai/carriage_right.obj
- link follower_right_link_1: geometry visual mesh filename=../meshes/wxai/link_1.obj
- link follower_right_link_2: geometry collision box size=0.3 0.05 0.05; visual mesh filename=../meshes/wxai/link_2.obj
- link follower_right_link_3: geometry collision box size=0.22 0.05 0.04; visual mesh filename=../meshes/wxai/link_3.obj
- link follower_right_link_4: geometry collision cylinder length=0.06 radius=0.029; visual mesh filename=../meshes/wxai/link_4.obj
- link follower_right_link_5: geometry collision cylinder length=0.05 radius=0.029; visual mesh filename=../meshes/wxai/link_5.obj
- link follower_right_link_6: geometry collision box size=0.025 0.187 0.0618; collision cylinder length=0.05 radius=0.029

Commit message: weld the table to the world

File: urdf/stationary_ai.urdf (robot description, URDF)
Before this commit: robot stationary_ai, 70 links, 69 joints
Joints:
- added joint world_joint: type fixed, parent world, child frame_link, origin xyz=0 0 0 rpy=0 0 0
